File: boards/esp8266-board/esp8266-board.brd (EAGLE design)
At the start: 24.9 x 40 mm, 16 parts, among them P1 ESP8266, P2 ESP8266 CONNECTOR, T1 AMS1117, T2 LM7805

Commit message: ESP8266 board updating
Parts:
- R1: device stutz-eagle:RESISTOR-V3 -> stutz-eagle:RESISTOR-V2
- moved C5 0.89 mm to (19.0, 3.91), turned to 270 degrees
- moved C4 0.64 mm to (21.1, 7.83)
- moved R1 0.32 mm to (19.9, 34.7)
Routing:
- net +3.3V: track 79.0 -> 73.6 mm
- net GND: track 113.0 -> 108.1 mm
- net ESP_RX: track 16.9 -> 14.6 mm
- net +5V: track 64.1 -> 64.9 mm
Other:
- board text added: "ESP8266"
- board text added: "FEMALE PIN"
- board text added: "LM7805"
- board text added: "SOLDERED"
