File: boards/esp8266-board/esp8266-board.sch (EAGLE design)
At the start: 16 parts, among them P1 ESP8266, P2 ESP8266 CONNECTOR, T1 AMS1117, T2 LM7805

Commit message: ESP8266 board updating
Parts:
- R1: device stutz-eagle:RESISTORV3 -> stutz-eagle:RESISTORV2
Changed lines of the file:
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@@
 <part name="U$3" library="stutz-eagle" deviceset="+24V" device=""/>
 <part name="SUPPLY11" library="stutz-eagle" deviceset="+3.3V" device=""/>
-<part name="R1" library="stutz-eagle" deviceset="RESISTOR" device="V3" value="3k3"/>
+<part name="R1" library="stutz-eagle" deviceset="RESISTOR" device="V2" value="3k3"/>
 </parts>
 <sheets>
