File: hardware/esp8266-12-board-v2.0/esp8266-board.brd (EAGLE design)
At the start: 35.4 x 38 mm, 24 parts, among them T1 AMS1117, T2 LM7805

Commit message: just after notebook crash
Parts:
- SD1: value CS SI GND 3.3V SCK GND SO -> SO GND SCK 3.3V GND SI CS
Changed lines of the file:
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@@
 </element>
 <element name="W1" library="stutz-eagle" package="SOT23-5/TSOT25" value="TPS3823-33" x="11" y="25.2" rot="MR0"/>
-<element name="SD1" library="stutz-eagle" package="PIN-HEADER-7PIN" value="CS  SI GND 3.3V SCK GND SO" x="1.7" y="18.9" smashed="yes" rot="R270">
-<attribute name="VALUE" x="4.333" y="27.99" size="0.9" layer="27" ratio="10" rot="R270"/>
+<element name="SD1" library="stutz-eagle" package="PIN-HEADER-7PIN" value="SO GND SCK 3.3V GND SI CS" x="1.7" y="18.9" smashed="yes" rot="R270">
+<attribute name="VALUE" x="4.333" y="26.99" size="0.9" layer="27" ratio="10" rot="R270"/>
 </element>
 </elements>
