File: hardware/esp8266-12-board-v2.0/esp8266-board.sch (EAGLE design)
At the start: 24 parts, among them T1 AMS1117, T2 LM7805

Commit message: just after notebook crash
Parts:
- SD1: value CS SI GND 3.3V SCK GND SO -> SO GND SCK 3.3V GND SI CS
- T2: device stutz-eagle:LM7805 -> stutz-components-library:LM7805
Changed lines of the file:
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@@
 <part name="C5" library="capacitor-wima" deviceset="C" device="2.5/2" value="10uF"/>
 <part name="U$1" library="stutz-eagle" deviceset="+24V" device=""/>
-<part name="T2" library="stutz-eagle" deviceset="LM7805" device="" value="LM7805">
+<part name="T2" library="stutz-components-library" deviceset="LM7805" device="" value="LM7805">
 <attribute name="MPN" value="LM2937ET-3.3"/>
 </part>
@@
 <part name="SUPPLY11" library="stutz-eagle" deviceset="+3.3V" device=""/>
 <part name="SUPPLY15" library="supply2" deviceset="GND" device=""/>
-<part name="SD1" library="stutz-eagle" deviceset="PIN-HEADER-7PIN" device="" value="CS  SI GND 3.3V SCK GND SO"/>
+<part name="SD1" library="stutz-eagle" deviceset="PIN-HEADER-7PIN" device="" value="SO GND SCK 3.3V GND SI CS"/>
 </parts>
 <sheets>
